File: PWM/GeraOndQuad_KiCad/GeraOndQuad.kicad_pcb (KiCad board)
At the start: 2 copper layers, 62.5 x 89.7 mm, 54 parts, among them U1 LM324, U2 TL494, U3 LM324, U4 TL494

Commit message: corrected kiCad errors
Parts:
- removed ANALOG-WAITER-ROBOT, AWR-19, JP1, JP2, JP5, JP6, JP7, JP8, JP9: Conn_01x01_Female, Connector_Wire:SolderWire-0.5sqmm_1x01_D0.9mm_OD2.1mm
- J1: renamed from GND | +5V | +12V | -12V
- J2: renamed from RMES | LMES
- J3: renamed from RPWM | LPWM
Routing:
- net Net-(R6L1-Pad2): vias 0 -> 2
- net GND: vias 0 -> 2
- net (no net): vias 0 -> 5
Other:
- board text added: "ANALOG WAITER ROBOT"
- board text added: "AWR - 19"
- board text added: "PWM"
