File: PWM/GeraOndQuad_KiCad/GeraOndQuad.kicad_pcb (KiCad board)
At the start: 2 copper layers, 62.5 x 89.7 mm, 45 parts, among them J1 Conn_01x04_Female, J2 Conn_01x02_Female, J3 Conn_01x02_Female, U1 LM324, U2 TL494, U3 LM324, U4 TL494

Commit message: GeraOndQuad Kicad name update
Parts:
- GND | +5V | +12V | -12V: renamed from J1
- RMES | LMES: renamed from J2
- RPWM | LPWM: renamed from J3
- moved RMES | LMES 0.51 mm to (64.8, 60.7)
Routing:
- net LMES: track 35.2 -> 37.8 mm
- net RMES: track 48.0 -> 50.0 mm
Other:
- board text added: "AWR-19_PWM"
- board text removed: "ANALOG WAITER ROBOT"
- board text removed: "AWR - 19"
- board text removed: "PWM"
