File: FSM/PCB_FSM_v1.8/KiCad/fsm.sch (KiCad schematic (older format))
At the start: 31 parts

Commit message: KiCad over
Parts:
- BRST1: footprint Connector_PinSocket_1.00mm:PinSocket_1x02_P1.00mm_Vertical -> Connector_PinSocket_2.00mm:PinSocket_1x02_P2.00mm_Vertical
Changed lines of the file:
@@
 F 0 "BRST1" H 2928 7076 50  0000 L CNN
 F 1 "Conn_01x02_Female" H 2928 6985 50  0001 L CNN
-F 2 "Connector_PinSocket_1.00mm:PinSocket_1x02_P1.00mm_Vertical" H 2900 7100 50  0001 C CNN
+F 2 "Connector_PinSocket_2.00mm:PinSocket_1x02_P2.00mm_Vertical" H 2900 7100 50  0001 C CNN
 F 3 "~" H 2900 7100 50  0001 C CNN
 	1    2900 7100
